File: my_anode/my_anode.kicad_pcb (KiCad board)
At the start: 2 copper layers, 326.8 x 374 mm, 133 parts, among them J1 7816-0000PR

Commit message: Add files via upload
Parts:
- moved J1 26.4 mm to (421.9, 488.4)
- moved GND2 18.8 mm to (217.4, 489.7), turned to 90 degrees
- moved BIAS1 16.7 mm to (365.8, 489.7), turned to 90 degrees
- moved GND1 14.4 mm to (286.8, 489.7), turned to 90 degrees
- moved SIG1 11.9 mm to (157.0, 490.0), turned to 90 degrees
- moved R23 5.99 mm to (339.1, 170.5)
- moved R25 5.99 mm to (331.5, 155.1)
- moved C9 5.99 mm to (353.1, 160.9)
- moved R21 5.99 mm to (348.2, 154.5)
- moved R22 5.99 mm to (339.3, 154.3)
- moved R24 5.99 mm to (331.7, 159.9)
- moved C10 5.99 mm to (332.0, 166.2)
- moved D5 5.99 mm to (342.6, 162.1)
Routing:
- net /S5: track 35.8 -> 587.6 mm, vias 0 -> 2
- net /B13: track 5.47 -> 552.5 mm, vias 0 -> 2
- net /1G13: track 12.6 -> 513.9 mm, vias 0 -> 2
- net /G9: track 40.5 -> 530.2 mm, vias 0 -> 2
- net /S6: track 27.9 -> 498.6 mm, vias 0 -> 4
- net /B9: track 9.59 -> 470.0 mm, vias 0 -> 2
- net /B14: track 17.6 -> 462.9 mm, vias 0 -> 2
- net /S7: track 24.9 -> 467.4 mm, vias 0 -> 4
- net /S9: track 27.9 -> 449.7 mm, vias 0 -> 2
- net /B5: track 11.7 -> 427.8 mm
- net /1G14: track 17.4 -> 431.1 mm, vias 0 -> 2
- net /G5: track 37.0 -> 431.0 mm, vias 0 -> 2
- net /B10: track 12.3 -> 396.3 mm, vias 0 -> 2
- net /G13: track 36.0 -> 418.6 mm, vias 0 -> 2
- net /1G9: track 15.4 -> 387.6 mm, vias 0 -> 2
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Other:
- board size 326.8 x 374 mm -> 327 x 404.6 mm

Commit message: Update anode work with mounting holes
Parts:
- added TP1: TestPoint, TestPoint:TestPoint_Loop_D3.80mm_Drill2.0mm, F.Cu at (184.5, 416.1)
- added TP10: TestPoint, TestPoint:TestPoint_Loop_D3.80mm_Drill2.0mm, F.Cu at (424.7, 335.4)
- added TP11: TestPoint, TestPoint:TestPoint_Loop_D3.80mm_Drill2.0mm, F.Cu at (424.9, 255.6)
- added TP12: TestPoint, TestPoint:TestPoint_Loop_D3.80mm_Drill2.0mm, F.Cu at (425.2, 169.5)
- added TP13: TestPoint, TestPoint:TestPoint_Loop_D3.80mm_Drill2.0mm, F.Cu at (343.1, 169.9)
- added TP14: TestPoint, TestPoint:TestPoint_Loop_D3.80mm_Drill2.0mm, F.Cu at (343.2, 255.8)
- added TP15: TestPoint, TestPoint:TestPoint_Loop_D3.80mm_Drill2.0mm, F.Cu at (343.0, 335.3)
- added TP16: TestPoint, TestPoint:TestPoint_Loop_D3.80mm_Drill2.0mm, F.Cu at (343.1, 416.1)
- added TP2: TestPoint, TestPoint:TestPoint_Loop_D3.80mm_Drill2.0mm, F.Cu at (184.1, 335.3)
- added TP3: TestPoint, TestPoint:TestPoint_Loop_D3.80mm_Drill2.0mm, F.Cu at (184.1, 255.6)
- added TP4: TestPoint, TestPoint:TestPoint_Loop_D3.80mm_Drill2.0mm, F.Cu at (184.4, 169.8)
- added TP5: TestPoint, TestPoint:TestPoint_Loop_D3.80mm_Drill2.0mm, F.Cu at (263.6, 416.2)
- added TP6: TestPoint, TestPoint:TestPoint_Loop_D3.80mm_Drill2.0mm, F.Cu at (263.6, 335.2)
- added TP7: TestPoint, TestPoint:TestPoint_Loop_D3.80mm_Drill2.0mm, F.Cu at (263.7, 255.8)
- added TP8: TestPoint, TestPoint:TestPoint_Loop_D3.80mm_Drill2.0mm, F.Cu at (263.5, 169.7)
- added TP9: TestPoint, TestPoint:TestPoint_Loop_D3.80mm_Drill2.0mm, B.Cu at (424.9, 415.9)
- moved C26 13.3 mm to (168.6, 165.2)
- moved R63 13.3 mm to (174.7, 167.0)
- moved C25 13.3 mm to (188.1, 157.8)
- moved D13 13.3 mm to (179.0, 159.6)
- moved R61 13.3 mm to (182.3, 151.5)
- moved R64 13.3 mm to (168.1, 158.6)
- moved R65 13.3 mm to (168.1, 155.6)
- moved R62 13.3 mm to (178.0, 151.0)
- moved C27 11.8 mm to (187.4, 242.4)
- moved C28 11.8 mm to (169.4, 254.6)
- moved D14 11.8 mm to (178.9, 245.5)
- moved R66 11.8 mm to (183.3, 237.6)
- moved R67 11.8 mm to (179.0, 237.6)
- moved R68 11.8 mm to (175.7, 253.3)
- moved R69 11.8 mm to (169.1, 247.0)
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Connections:
- J1 pad 1: unconnected-(J1-Pad1) -> Net-(J1-Pad1)
- J1 pad 10: unconnected-(J1-Pad10) -> Net-(J1-Pad10)
- J1 pad 11: unconnected-(J1-Pad11) -> Net-(J1-Pad11)
- J1 pad 12: unconnected-(J1-Pad12) -> Net-(J1-Pad12)
- J1 pad 13: unconnected-(J1-Pad13) -> Net-(J1-Pad13)
- J1 pad 14: unconnected-(J1-Pad14) -> Net-(J1-Pad14)
- J1 pad 15: unconnected-(J1-Pad15) -> Net-(J1-Pad15)
- J1 pad 16: unconnected-(J1-Pad16) -> Net-(J1-Pad16)
- J1 pad 2: unconnected-(J1-Pad2) -> Net-(J1-Pad2)
- J1 pad 3: unconnected-(J1-Pad3) -> Net-(J1-Pad3)
- J1 pad 4: unconnected-(J1-Pad4) -> Net-(J1-Pad4)
- J1 pad 5: unconnected-(J1-Pad5) -> Net-(J1-Pad5)
- J1 pad 6: unconnected-(J1-Pad6) -> Net-(J1-Pad6)
- J1 pad 7: unconnected-(J1-Pad7) -> Net-(J1-Pad7)
- J1 pad 8: unconnected-(J1-Pad8) -> Net-(J1-Pad8)
- J1 pad 9: unconnected-(J1-Pad9) -> Net-(J1-Pad9)
Routing:
- net Net-(J1-Pad1): track 0.00 -> 1018.2 mm
- net unconnected-(J1-Pad1): track 939.9 -> 0.00 mm, vias 1 -> 0
- net Net-(J1-Pad3): track 0.00 -> 910.8 mm
- net Net-(J1-Pad9): track 0.00 -> 906.8 mm
- net unconnected-(J1-Pad3): track 853.0 -> 0.00 mm, vias 1 -> 0
- net unconnected-(J1-Pad9): track 819.4 -> 0.00 mm, vias 1 -> 0
- net Net-(J1-Pad5): track 0.00 -> 802.3 mm
- net Net-(J1-Pad11): track 0.00 -> 795.9 mm
- net Net-(J1-Pad16): track 0.00 -> 782.4 mm
- net unconnected-(J1-Pad5): track 758.3 -> 0.00 mm, vias 1 -> 0
- net unconnected-(J1-Pad11): track 731.6 -> 0.00 mm, vias 1 -> 0
- net Net-(J1-Pad7): track 0.00 -> 689.6 mm
- net Net-(J1-Pad13): track 0.00 -> 689.6 mm
- net unconnected-(J1-Pad16): track 687.2 -> 0.00 mm, vias 1 -> 0
- net Net-(J1-Pad14): track 0.00 -> 678.7 mm
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Other:
- board size 327 x 404.6 mm -> 326.8 x 407.5 mm

Commit message: Add quarter-anode board
Parts:
- removed BIAS1, GND1, GND2, J1, SIG1: 7816-0000PR, 7816-0000PR:3M_7816-0000PR
- removed C10, C11, C12, C13, C14, C15, C16, C17, C18, C19, C20, C21, C22, C23, C24, C25, C26, C27, C28, C29, C30, C31, C32, C9: C, Capacitor_SMD:CP_Elec_4x3
- removed D10, D11, D12, D13, D14, D15, D16, D5, D6, D7, D8, D9: D_Photo, OptoDevice:S13370-6075CN
- removed R21, R22, R23, R24, R25, R26, R27, R28, R29, R30, R31, R32, R33, R34, R35, R36, R37, R38, R39, R40, R41, R42, R43, R44, R45, R46, R47, R48, R49, R50, R51, R52, R53, R54, R55, R56, R57, R58, R59, R60, R61, R62, R63, R64, R65, R66, R67, R68, R69, R70, R71, R72, R73, R74, R75, R76, R77, R78, R79, R80: R_US, Resistor_SMD:R_0402_1005Metric
- removed TP10, TP11, TP12, TP13, TP14, TP15, TP16, TP5, TP6, TP7, TP8, TP9: TestPoint, TestPoint:TestPoint_Loop_D3.80mm_Drill2.0mm
- added J3: 430451019, footprints:430451019, F.Cu at (186.5, 188.5)
- added J4: CON_430450419_MOL, 430450419:430450419, F.Cu at (234.1, 199.2)
- added MOUNTING: MountingHole_2.1mm, MountingHole:MountingHole_2.1mm, F.Cu at (190.2, 210.1)
- added REF**: MountingHole_2.1mm, MountingHole:MountingHole_2.1mm, F.Cu at (281.2, 157.8)
- added REF**: MountingHole_2.1mm, MountingHole:MountingHole_2.1mm, F.Cu at (161.0, 119.2)
- added REF**: MountingHole_2.1mm, MountingHole:MountingHole_2.1mm, F.Cu at (201.8, 119.2)
- added REF**: MountingHole_2.1mm, MountingHole:MountingHole_2.1mm, F.Cu at (281.1, 239.4)
- added REF**: MountingHole_2.1mm, MountingHole:MountingHole_2.1mm, F.Cu at (242.5, 119.2)
- added REF**: MountingHole_2.1mm, MountingHole:MountingHole_2.1mm, F.Cu at (281.1, 198.6)
- C1, C2, C3, C4, C5, C6, C7, C8: footprint Capacitor_SMD:CP_Elec_4x3 -> Capacitor_SMD:C_1812_4532Metric_Pad1.57x3.40mm_HandSolder
- moved C4 313.7 mm to (160.2, 141.4), turned to 0 degrees
- moved C2 313.6 mm to (241.6, 148.4), turned to 180 degrees
- moved R8 313.1 mm to (162.9, 146.3), turned to 0 degrees
- moved R3 313.0 mm to (247.7, 149.9), turned to 180 degrees
- moved R5 312.1 mm to (241.9, 143.5), turned to 180 degrees
- moved R10 310.3 mm to (160.7, 135.8), turned to 180 degrees
- moved C3 310.1 mm to (160.2, 167.2), turned to 180 degrees
- moved C1 309.6 mm to (233.9, 163.7), turned to 0 degrees
- moved R9 308.7 mm to (158.3, 147.4), turned to -90 degrees
- moved D2 308.2 mm to (161.2, 156.7), turned to 90 degrees
- moved R4 306.6 mm to (247.6, 143.2), turned to 0 degrees
- moved R1 305.9 mm to (228.7, 161.5), turned to 0 degrees
- moved D1 304.5 mm to (242.9, 157.5)
- moved R6 297.5 mm to (166.5, 168.4), turned to -90 degrees
- moved R2 294.5 mm to (231.5, 168.2), turned to 0 degrees
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Connections:
- C4 pad 2: /1G2 -> /1G1
- C6 pad 2: /1G3 -> /1G1
- C8 pad 2: /1G4 -> /1G1
- R10 pad 1: /B2 -> /B1
- R13 pad 2: /1G3 -> /1G1
- R15 pad 1: /B3 -> /B1
- R18 pad 2: /1G4 -> /1G1
- R20 pad 1: /B4 -> /B1
- R8 pad 2: /1G2 -> /1G1
Routing:
- net Net-(J4-Pad1): track 1018.2 -> 30.5 mm
- net Net-(J1-Pad9): track 906.8 -> 0.00 mm
- net Net-(J4-Pad2): track 910.8 -> 77.4 mm
- net Net-(J1-Pad11): track 795.9 -> 0.00 mm
- net Net-(J1-Pad16): track 782.4 -> 0.00 mm
- net Net-(TP3-Pad1): track 802.3 -> 89.7 mm
- net Net-(J1-Pad13): track 689.6 -> 0.00 mm
- net Net-(J1-Pad14): track 678.7 -> 0.00 mm
- net Net-(J4-Pad4): track 689.6 -> 33.6 mm
- net /S5: track 587.6 -> 0.00 mm, vias 2 -> 0
- net Net-(J1-Pad12): track 576.4 -> 0.00 mm
- net Net-(J1-Pad15): track 563.0 -> 0.00 mm
- net /B13: track 556.7 -> 0.00 mm, vias 2 -> 0
- net /S3: track 583.3 -> 45.6 mm, vias 2 -> 0
- net /1G13: track 520.0 -> 0.00 mm, vias 2 -> 0
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Other:
- board size 326.8 x 407.5 mm -> 163 x 163 mm

Commit message: Semi-final board version without voltage divider
Parts:
- removed TP1, TP2, TP3, TP4: TestPoint, TestPoint:TestPoint_Loop_D3.80mm_Drill2.0mm
- J4: value CON_430450419_MOL -> 430450419
- moved J3 27.8 mm to (211.9, 177.2)
- moved C7 19.6 mm to (250.6, 229.2)
- moved R16 18.7 mm to (244.9, 228.7), turned to 180 degrees
- moved R19 17.5 mm to (255.0, 243.4)
- moved J4 11.7 mm to (234.5, 187.5)
- turned D1 to 180 degrees
- turned D2 to -90 degrees
- turned D4 to 90 degrees
Connections:
- D1 pad 1: /G1 -> Net-(C1-Pad2)
- D1 pad 2: Net-(C1-Pad2) -> /G1
- D2 pad 1: /G2 -> Net-(C3-Pad2)
- D2 pad 2: Net-(C3-Pad2) -> /G2
- D3 pad 1: /G3 -> Net-(C5-Pad2)
- D3 pad 2: Net-(C5-Pad2) -> /G3
- D4 pad 1: /G4 -> Net-(C7-Pad2)
- D4 pad 2: Net-(C7-Pad2) -> /G4
- J4 pad 1: Net-(J4-Pad1) -> zone1
- J4 pad 2: Net-(J4-Pad2) -> zone2
- J4 pad 3: Net-(TP3-Pad1) -> zone3
- J4 pad 4: Net-(J4-Pad4) -> zone4
- R14 pad 2: /G3 -> Net-(C5-Pad2)
- R19 pad 2: /G4 -> Net-(C7-Pad2)
- R4 pad 2: /G1 -> Net-(C1-Pad2)
- R9 pad 2: /G2 -> Net-(C3-Pad2)
Routing:
- net /G4: track 269.5 -> 149.5 mm
- net /S4: track 231.2 -> 117.2 mm
- net zone3: track 0.00 -> 96.0 mm, vias 0 -> 1
- net /B1: track 564.3 -> 472.4 mm
- net Net-(TP3-Pad1): track 89.7 -> 0.00 mm
- net /S1: track 113.7 -> 29.7 mm
- net /G1: track 149.8 -> 67.6 mm
- net Net-(J4-Pad2): track 77.4 -> 0.00 mm
- net zone2: track 0.00 -> 73.8 mm, vias 0 -> 1
- net zone4: track 0.00 -> 45.5 mm, vias 0 -> 1
- net Net-(C5-Pad2): track 14.4 -> 49.6 mm
- net Net-(J4-Pad4): track 33.6 -> 0.00 mm
- net Net-(J4-Pad1): track 30.5 -> 0.00 mm
- net /S2: track 45.2 -> 73.9 mm
- net /S3: track 45.6 -> 72.1 mm
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- added copper zone on B.Cu, net zone1
- added copper zone on B.Cu, net zone2
- added copper zone on B.Cu, net zone3
- added copper zone on B.Cu, net zone4
- removed copper zone on B.Cu, net (none)

Commit message: Add files via upload
Parts:
- added R21: R_US, Resistor_SMD:R_0402_1005Metric, F.Cu at (228.2, 240.2)
- added R22: R_Variable_US, Potentiometer_SMD:Potentiometer_Bourns_3214G_Horizontal, F.Cu at (212.6, 256.1)
- added R23: R_US, Resistor_SMD:R_0402_1005Metric, F.Cu at (237.1, 137.7)
- added R24: R_Variable_US, Potentiometer_SMD:Potentiometer_Bourns_3214G_Horizontal, F.Cu at (221.2, 142.0)
- added R25: R_US, Resistor_SMD:R_0402_1005Metric, F.Cu at (192.4, 136.3)
- added R26: R_Variable_US, Potentiometer_SMD:Potentiometer_Bourns_3214G_Horizontal, F.Cu at (183.4, 141.7)
- added R27: R_US, Resistor_SMD:R_0402_1005Metric, F.Cu at (179.3, 257.6)
- added R28: R_Variable_US, Potentiometer_SMD:Potentiometer_Bourns_3214G_Horizontal, F.Cu at (190.7, 256.7)
- moved R10 10.3 mm to (163.5, 145.8)
- moved R8 10.2 mm to (172.5, 149.9)
Connections:
- net zone1 renamed Net-(J4-Pad1)
- net zone2 renamed Net-(J4-Pad2)
- net zone3 renamed Net-(J4-Pad3)
- net zone4 renamed Net-(J4-Pad4)
- R10 pad 1: /B1 -> Net-(R10-Pad1)
- R15 pad 1: /B1 -> Net-(R15-Pad1)
- R20 pad 1: /B1 -> Net-(R20-Pad1)
- R5 pad 1: /B1 -> Net-(R5-Pad1)
Routing:
- net /1G1: track 345.4 -> 500.4 mm
- net /B1: track 472.4 -> 321.5 mm
- net Net-(R20-Pad1): track 0.00 -> 96.1 mm
- net Net-(R10-Pad1): track 0.00 -> 33.4 mm
- net Net-(R5-Pad1): track 0.00 -> 29.6 mm
- net Net-(R15-Pad1): track 0.00 -> 24.9 mm
- net Net-(C4-Pad1): track 12.0 -> 13.6 mm
